File: Board/RAMPS_FanSpansion.brd (EAGLE design)
At the start: 18.5 x 22 mm, 19 parts

Commit message: Exported PDFs
Routing:
- net N$9: track 0.00 -> 1.00 mm
- net N$8: track 0.00 -> 1.00 mm
- net N$7: track 0.00 -> 1.00 mm
- net N$5: track 0.00 -> 1.00 mm
- net N$21: track 0.00 -> 1.00 mm
- net N$20: track 0.00 -> 1.00 mm
- net N$19: track 0.00 -> 1.00 mm
- net N$18: track 0.00 -> 1.00 mm
- net N$17: track 0.00 -> 1.00 mm
- net N$16: track 0.00 -> 1.00 mm
- net N$15: track 0.00 -> 1.00 mm
- net N$14: track 0.00 -> 1.00 mm
- net N$13: track 0.00 -> 1.00 mm
- net N$12: track 0.00 -> 1.00 mm
- net N$11: track 0.00 -> 1.00 mm
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Changed lines of the file:
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@@
 </autorouter>
 <elements>
-<element name="D1" library="diode" package="SOD323-R" value="1n4148" x="1.905" y="2.54" rot="R90"/>
-<element name="D2" library="diode" package="SOD323-R" value="1n4148" x="1.905" y="6.35" rot="R90"/>
-<element name="D3" library="diode" package="SOD323-R" value="1n4148" x="17.145" y="2.54" rot="R90"/>
-<element name="D4" library="diode" package="SOD323-R" value="1n4148" x="17.145" y="6.35" rot="R90"/>
-<element name="JP1" library="pinhead" package="2X03" value="" x="13.335" y="17.78" rot="R90"/>
-<element name="JP2" library="pinhead" package="2X03" value="" x="8.255" y="17.78" rot="R90"/>
-<element name="JP3" library="pinhead" package="2X05" value="" x="9.525" y="3.175" rot="R180"/>
-<element name="JP4" library="pinhead" package="1X02" value="" x="3.175" y="16.51"/>
-<element name="LED1" library="led" package="SML0805" value="" x="6.985" y="11.43" rot="R90"/>
-<element name="LED2" library="led" package="SML0805" value="" x="9.525" y="11.43" rot="R90"/>
-<element name="LED3" library="led" package="SML0805" value="" x="12.065" y="11.43" rot="R90"/>
-<element name="LED4" library="led" package="SML0805" value="" x="14.605" y="11.43" rot="R90"/>
-<element name="R1" library="resistor" package="R0805" value="" x="6.985" y="7.62" rot="R90"/>
-<element name="R2" library="resistor" package="R0805" value="" x="9.525" y="7.62" rot="R90"/>
-<element name="R3" library="resistor" package="R0805" value="" x="12.065" y="7.62" rot="R90"/>
-<element name="R4" library="resistor" package="R0805" value="" x="14.605" y="7.62" rot="R90"/>
-<element name="U$1" library="RobThePyro" package="SO08" value="DMG4800LSD" x="8.255" y="9.525" rot="MR180"/>
-<element name="U$2" library="RobThePyro" package="SO08" value="DMG4800LSD" x="13.335" y="9.525" rot="MR180"/>
-<element name="F1" library="adafruit" package="1812" value="" x="1.905" y="11.43" rot="MR90"/>
+<element name="D1" library="diode" package="SOD323-R" value="1n4148" x="1.905" y="2.54" smashed="yes" rot="R90"/>
+<element name="D2" library="diode" package="SOD323-R" value="1n4148" x="1.905" y="6.35" smashed="yes" rot="R90"/>
+<element name="D3" library="diode" package="SOD323-R" value="1n4148" x="17.145" y="2.54" smashed="yes" rot="R90"/>
+<element name="D4" library="diode" package="SOD323-R" value="1n4148" x="17.145" y="6.35" smashed="yes" rot="R90"/>
+<element name="JP1" library="pinhead" package="2X03" value="" x="13.335" y="17.78" smashed="yes" rot="R90">
+<attribute name="VALUE" x="17.78" y="13.97" size="1.27" layer="27" rot="R90"/>
+</element>
+<element name="JP2" library="pinhead" package="2X03" value="" x="8.255" y="17.78" smashed="yes" rot="R90">
+<attribute name="NAME" x="5.08" y="13.97" size="1.27" layer="25" ratio="10" rot="R90"/>
+<attribute name="VALUE" x="12.7" y="13.97" size="1.27" layer="27" rot="R90"/>
+</element>
+<element name="JP3" library="pinhead" package="2X05" value="" x="9.525" y="3.175" smashed="yes" rot="R180">
+<attribute name="VALUE" x="15.875" y="7.62" size="1.27" layer="27" rot="R180"/>
+</element>
+<element name="JP4" library="pinhead" package="1X02" value="" x="3.175" y="16.51" smashed="yes">
+<attribute name="VALUE" x="0.635" y="13.335" size="1.27" layer="27"/>
+</element>
+<element name="LED1" library="led" package="SML0805" value="" x="6.985" y="11.43" smashed="yes" rot="R90">
+<attribute name="VALUE" x="8.985" y="9.93" size="1.27" layer="27" rot="R90"/>
+</element>
+<element name="LED2" library="led" package="SML0805" value="" x="9.525" y="11.43" smashed="yes" rot="R90">
+<attribute name="VALUE" x="11.525" y="9.93" size="1.27" layer="27" rot="R90"/>
+</element>
+<element name="LED3" library="led" package="SML0805" value="" x="12.065" y="11.43" smashed="yes" rot="R90">
+<attribute name="VALUE" x="14.065" y="9.93" size="1.27" layer="27" rot="R90"/>
+</element>
+<element name="LED4" library="led" package="SML0805" value="" x="14.605" y="11.43" smashed="yes" rot="R90">
+<attribute name="VALUE" x="16.605" y="9.93" size="1.27" layer="27" rot="R90"/>
+</element>
+<element name="R1" library="resistor" package="R0805" value="" x="6.985" y="7.62" smashed="yes" rot="R90">
+<attribute name="VALUE" x="9.525" y="6.985" size="1.27" layer="27" rot="R90"/>
+</element>
+<element name="R2" library="resistor" package="R0805" value="" x="9.525" y="7.62" smashed="yes" rot="R90">
+<attribute name="VALUE" x="12.065" y="6.985" size="1.27" layer="27" rot="R90"/>
+</element>
+<element name="R3" library="resistor" package="R0805" value="" x="12.065" y="7.62" smashed="yes" rot="R90">
+<attribute name="VALUE" x="14.605" y="6.985" size="1.27" layer="27" rot="R90"/>
+</element>
+<element name="R4" library="resistor" package="R0805" value="" x="14.605" y="7.62" smashed="yes" rot="R90">
+<attribute name="VALUE" x="17.145" y="6.985" size="1.27" layer="27" rot="R90"/>
+</element>
+<element name="U$1" library="RobThePyro" package="SO08" value="DMG4800LSD" x="8.255" y="9.525" smashed="yes" rot="MR180"/>
+<element name="U$2" library="RobThePyro" package="SO08" value="DMG4800LSD" x="13.335" y="9.525" smashed="yes" rot="MR180"/>
+<element name="F1" library="adafruit" package="1812" value="" x="1.905" y="11.43" smashed="yes" rot="MR90">
+<attribute name="VALUE" x="3.81" y="9.5725" size="0.6096" layer="28" rot="MR90"/>
+</element>
 </elements>
 <signals>
@@
 <wire x1="1.905" y1="16.51" x2="1.905" y2="13.476" width="1.27" layer="16"/>
 </signal>
+<signal name="N$5">
+<wire x1="0" y1="-0.5" x2="0" y2="0.5" width="0.3048" layer="16"/>
+</signal>
+<signal name="N$7">
+<wire x1="-0.5" y1="0" x2="0.5" y2="0" width="0.3048" layer="16"/>
+</signal>
+<signal name="N$8">
+<wire x1="18" y1="0" x2="19" y2="0" width="0.3048" layer="16"/>
+</signal>
+<signal name="N$9">
+<wire x1="18.5" y1="-0.5" x2="18.5" y2="0.5" width="0.3048" layer="16"/>
+</signal>
+<signal name="N$10">
+<wire x1="18.5" y1="22.5" x2="18.5" y2="21.5" width="0.3048" layer="16"/>
+</signal>
+<signal name="N$11">
+<wire x1="18" y1="22" x2="19" y2="22" width="0.3048" layer="16"/>
+</signal>
+<signal name="N$12">
+<wire x1="0" y1="22.5" x2="0" y2="21.5" width="0.3048" layer="16"/>
+</signal>
+<signal name="N$13">
+<wire x1="-0.5" y1="22" x2="0.5" y2="22" width="0.3048" layer="16"/>
+</signal>
+<signal name="N$14">
+<wire x1="0" y1="22.5" x2="0" y2="21.5" width="0.3048" layer="1"/>
+</signal>
+<signal name="N$15">
+<wire x1="-0.5" y1="22" x2="0.5" y2="22" width="0.3048" layer="1"/>
+</signal>
+<signal name="N$16">
+<wire x1="18.5" y1="22.5" x2="18.5" y2="21.5" width="0.3048" layer="1"/>
+</signal>
+<signal name="N$17">
+<wire x1="19" y1="22" x2="18" y2="22" width="0.3048" layer="1"/>
+</signal>
+<signal name="N$18">
+<wire x1="18.5" y1="0.5" x2="18.5" y2="-0.5" width="0.3048" layer="1"/>
+</signal>
+<signal name="N$19">
+<wire x1="18" y1="0" x2="19" y2="0" width="0.3048" layer="1"/>
+</signal>
+<signal name="N$20">
+<wire x1="0" y1="0.5" x2="0" y2="-0.5" width="0.3048" layer="1"/>
+</signal>
+<signal name="N$21">
+<wire x1="-0.5" y1="0" x2="0.5" y2="0" width="0.3048" layer="1"/>
+</signal>
 </signals>
